File: hw/controller/controller.sch (KiCad schematic (older format))
At the start: 57 parts, among them J1 ARM-SWD, P1 USB_OTG, P10 GPIO, P11 VDD_SEL, P12 UART0, P13 SPI, P14 I2C0, P15 I2C1, P16 I2C2, P17 I2C3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

Commit message: Updating part numbers for ostur controller
Parts:
- C1: MPN (none) -> CL21B104MBCNNNC; mpn CL21B103KBANNNC -> (none)
- C10, C6: MPN (none) -> CL21B104MBCNNNC
- C11, C2, C4: MPN (none) -> CL21B103KBANNNC
- C12, C13: MPN (none) -> CL10C120JB8NNNC
- C5: MPN (none) -> CL21B104MBCNNNC; mpn CL21B104MBCNNNC -> (none)
- C7, C9: MPN (none) -> CL21A475KQFNNNG
- C8: MPN (none) -> CL21F105ZAFNNNG
- D1, D2, D3: MPN (none) -> LG R971-KN-1
- J1: MPN (none) -> 20021121-00010C4LF
- P1: MPN (none) -> 10118192-0001LF; mpn 10118192-0001LF -> (none)
- R1: MPN (none) -> MCR10ERTJ000
- R10, R11, R12, R13, R14, R2, R21, R22, R23, R24: MPN (none) -> 311-10KARCT-ND
- R3: MPN (none) -> RC0805JR-07680RL; mpn RC0805JR-07680RL -> (none)
- R4, R5: MPN (none) -> RC0805JR-07680RL
- R6: MPN (none) -> RC0805JR-071K5L; mpn RC0805JR-071K5L -> (none)
- R7: MPN (none) -> RC0805JR-0722RL; mpn RC0805JR-0722RL -> (none)
- R8: MPN (none) -> RC0805JR-0722RL
- R9: MPN (none) -> 311-10KARCT-ND; mpn 311-10KARCT-ND -> (none)
- SW1: MPN (none) -> PTS645SM43SMTR92; mpn PTS645SM43SMTR92 -> (none)
- SW2: MPN (none) -> PTS645SM43SMTR92
- U1: MPN (none) -> STM32F072CBT6; mpn STM32F072CBT6 -> (none)
- U2: MPN (none) -> LD1117S33CTR; mpn LD1117S33CTR -> (none)
- U3: MPN (none) -> TCA9546APWR
- Y2: MPN (none) -> FC-135 32.7680KA-A0
Changed lines of the file:
@@
 F 2 "footprints:LQFP48" H 2000 2700 60  0001 C CNN
 F 3 "" H 2000 2700 60  0000 C CNN
-F 4 "STM32F072CBT6" H 2000 2700 60  0001 C CNN "mpn"
+F 4 "STM32F072CBT6" H 2000 2700 60  0001 C CNN "MPN"
 	1    2000 2700
 	1    0    0    -1
@@
 F 2 "Capacitors_SMD:C_0805" H 1700 1250 50  0001 C CNN
 F 3 "" H 1700 1250 50  0000 C CNN
-F 4 "CL21B104MBCNNNC" H 1700 1250 60  0001 C CNN "mpn"
+F 4 "CL21B104MBCNNNC" H 1700 1250 60  0001 C CNN "MPN"
 	1    1700 1250
 	1    0    0    -1
@@
 F 2 "Capacitors_SMD:C_0805" H 2000 1250 50  0001 C CNN
 F 3 "" H 2000 1250 50  0000 C CNN
+F 4 "CL21B104MBCNNNC" H 2000 1250 60  0001 C CNN "MPN"
 	1    2000 1250
 	1    0    0    -1
@@
 F 2 "Capacitors_SMD:C_0805" H 2300 1250 50  0001 C CNN
 F 3 "" H 2300 1250 50  0000 C CNN
+F 4 "CL21A475KQFNNNG" H 2300 1250 60  0001 C CNN "MPN"
 	1    2300 1250
 	1    0    0    -1
@@
 F 2 "Capacitors_SMD:C_0805" H 2600 1250 50  0001 C CNN
 F 3 "" H 2600 1250 50  0000 C CNN
+F 4 "CL21F105ZAFNNNG" H 2600 1250 60  0001 C CNN "MPN"
 	1    2600 1250
 	1    0    0    -1
@@
 F 2 "Capacitors_SMD:C_0805" H 1450 1250 50  0001 C CNN
 F 3 "" H 1450 1250 50  0000 C CNN
+F 4 "CL21B103KBANNNC" H 1450 1250 60  0001 C CNN "MPN"
 	1    1450 1250
 	1    0    0    -1
@@
 F 2 "footprints:PTS645SM43SMTR92" H 1700 6350 50  0001 C CNN
 F 3 "" H 1700 6350 50  0000 C CNN
-F 4 "PTS645SM43SMTR92" H 1700 6350 60  0001 C CNN "mpn"
+F 4 "PTS645SM43SMTR92" H 1700 6350 60  0001 C CNN "MPN"
 	1    1700 6350
 	1    0    0    -1
@@
 F 2 "footprints:PTS645SM43SMTR92" H 1700 6750 50  0001 C CNN
 F 3 "" H 1700 6750 50  0000 C CNN
+F 4 "PTS645SM43SMTR92" H 1700 6750 60  0001 C CNN "MPN"
 	1    1700 6750
 	1    0    0    -1
@@
 F 2 "Resistors_SMD:R_0805" V 2030 6950 50  0001 C CNN
 F 3 "" H 2100 6950 50  0000 C CNN
+F 4 "311-10KARCT-ND" V 2100 6950 60  0001 C CNN "MPN"
 	1    2100 6950
 	-1   0    0    1
@@
 F 2 "Capacitors_SMD:C_0805" H 2900 1250 50  0001 C CNN
 F 3 "" H 2900 1250 50  0000 C CNN
+F 4 "CL21A475KQFNNNG" H 2900 1250 60  0001 C CNN "MPN"
 	1    2900 1250
 	1    0    0    -1
@@
 F 2 "Capacitors_SMD:C_0805" H 1200 1250 50  0001 C CNN
 F 3 "" H 1200 1250 50  0000 C CNN
-F 4 "CL21B103KBANNNC" H 1200 1250 60  0001 C CNN "mpn"
+F 4 "CL21B104MBCNNNC" H 1200 1250 60  0001 C CNN "MPN"
 	1    1200 1250
 	1    0    0    -1
@@
 F 2 "LEDs:LED_0805" H 3600 7150 50  0001 C CNN
 F 3 "" H 3600 7150 50  0000 C CNN
+F 4 "LG R971-KN-1" H 3600 7150 60  0001 C CNN "MPN"
 	1    3600 7150
 	-1   0    0    1
@@
 F 2 "LEDs:LED_0805" H 3600 6850 50  0001 C CNN
 F 3 "" H 3600 6850 50  0000 C CNN
+F 4 "LG R971-KN-1" H 3600 6850 60  0001 C CNN "MPN"
 	1    3600 6850
 	-1   0    0    1
@@
 F 2 "LEDs:LED_0805" H 3600 6550 50  0001 C CNN
 F 3 "" H 3600 6550 50  0000 C CNN
+F 4 "LG R971-KN-1" H 3600 6550 60  0001 C CNN "MPN"
 	1    3600 6550
 	-1   0    0    1
@@
 F 2 "Resistors_SMD:R_0805" V 3080 7150 50  0001 C CNN
 F 3 "" H 3150 7150 50  0000 C CNN
+F 4 "RC0805JR-07680RL" V 3150 7150 60  0001 C CNN "MPN"
 	1    3150 7150
 	0    1    1    0
@@
 F 2 "Resistors_SMD:R_0805" V 3080 6850 50  0001 C CNN
 F 3 "" H 3150 6850 50  0000 C CNN
+F 4 "RC0805JR-07680RL" V 3150 6850 60  0001 C CNN "MPN"
 	1    3150 6850
 	0    1    1    0
@@
 F 2 "Resistors_SMD:R_0805" V 3080 6550 50  0001 C CNN
 F 3 "" H 3150 6550 50  0000 C CNN
-F 4 "RC0805JR-07680RL" V 3150 6550 60  0001 C CNN "mpn"
+F 4 "RC0805JR-07680RL" V 3150 6550 60  0001 C CNN "MPN"
 	1    3150 6550
 	0    1    1    0
@@
 F 2 "footprints:FC-135" H 5000 4600 50  0001 C CNN
 F 3 "" H 5000 4600 50  0000 C CNN
+F 4 "FC-135 32.7680KA-A0" H 5000 4600 60  0001 C CNN "MPN"
 	1    5000 4600
 	0    -1   -1   0
@@
 F 2 "Capacitors_SMD:C_0603" H 5300 4800 50  0001 C CNN
 F 3 "" H 5300 4800 50  0000 C CNN
+F 4 "CL10C120JB8NNNC" H 5300 4800 60  0001 C CNN "MPN"
 	1    5300 4800
 	0    -1   -1   0
@@
 F 2 "Capacitors_SMD:C_0603" H 5300 4400 50  0001 C CNN
 F 3 "" H 5300 4400 50  0000 C CNN
+F 4 "CL10C120JB8NNNC" H 5300 4400 60  0001 C CNN "MPN"
 	1    5300 4400
 	0    -1   -1   0
@@
 F 2 "footprints:USB_MICRO_B" V 6150 6750 50  0001 C CNN
 F 3 "" V 6150 6750 50  0000 C CNN
-F 4 "10118192-0001LF" H 6200 6850 60  0001 C CNN "mpn"
+F 4 "10118192-0001LF" H 6200 6850 60  0001 C CNN "MPN"
 	1    6200 6850
 	0    1    1    0
@@
 F 2 "Resistors_SMD:R_0805" V 5380 6750 50  0001 C CNN
 F 3 "" H 5450 6750 50  0000 C CNN
-F 4 "RC0805JR-0722RL" V 5450 6750 60  0001 C CNN "mpn"
+F 4 "RC0805JR-0722RL" V 5450 6750 60  0001 C CNN "MPN"
 	1    5450 6750
 	0    1    1    0
@@
 F 2 "Resistors_SMD:R_0805" V 5380 6950 50  0001 C CNN
 F 3 "" H 5450 6950 50  0000 C CNN
+F 4 "RC0805JR-0722RL" V 5450 6950 60  0001 C CNN "MPN"
 	1    5450 6950
 	0    1    1    0
@@
 F 2 "Resistors_SMD:R_0805" V 5030 7200 50  0001 C CNN
 F 3 "" H 5100 7200 50  0000 C CNN
-F 4 "RC0805JR-071K5L" V 5100 7200 60  0001 C CNN "mpn"
+F 4 "RC0805JR-071K5L" V 5100 7200 60  0001 C CNN "MPN"
 	1    5100 7200
 	-1   0    0    1
@@
 F 2 "footprints:SOT-223" H 4200 1250 50  0001 C CNN
 F 3 "" H 4200 1150 50  0000 C CNN
-F 4 "LD1117S33CTR" H 4200 1150 60  0001 C CNN "mpn"
+F 4 "LD1117S33CTR" H 4200 1150 60  0001 C CNN "MPN"
 	1    4200 1150
 	1    0    0    -1
@@
 F 2 "Capacitors_SMD:C_0805" H 3550 1250 50  0001 C CNN
 F 3 "" H 3550 1250 50  0000 C CNN
+F 4 "CL21B104MBCNNNC" H 3550 1250 60  0001 C CNN "MPN"
 	1    3550 1250
 	1    0    0    -1
@@
 F 2 "Capacitors_SMD:C_0805" H 4850 1250 50  0001 C CNN
 F 3 "" H 4850 1250 50  0000 C CNN
+F 4 "CL21B103KBANNNC" H 4850 1250 60  0001 C CNN "MPN"
 	1    4850 1250
 	1    0    0    -1
@@
 F 2 "Resistors_SMD:R_0805" V 9930 1200 50  0001 C CNN
 F 3 "" H 10000 1200 50  0000 C CNN
+F 4 "311-10KARCT-ND" V 10000 1200 60  0001 C CNN "MPN"
 	1    10000 1200
 	0    -1   -1   0
@@
 F 2 "Resistors_SMD:R_0805" V 9930 1350 50  0001 C CNN
 F 3 "" H 10000 1350 50  0000 C CNN
+F 4 "311-10KARCT-ND" V 10000 1350 60  0001 C CNN "MPN"
 	1    10000 1350
 	0    -1   -1   0
@@
 F 2 "Resistors_SMD:R_0805" V 9930 850 50  0001 C CNN
 F 3 "" H 10000 850 50  0000 C CNN
-F 4 "311-10KARCT-ND" V 10000 850 60  0001 C CNN "mpn"
+F 4 "311-10KARCT-ND" V 10000 850 60  0001 C CNN "MPN"
 	1    10000 850
 	0    -1   -1   0
@@
 F 2 "Resistors_SMD:R_0805" V 9930 1000 50  0001 C CNN
 F 3 "" H 10000 1000 50  0000 C CNN
+F 4 "311-10KARCT-ND" V 10000 1000 60  0001 C CNN "MPN"
 	1    10000 1000
 	0    -1   -1   0
@@
 F 2 "Resistors_SMD:R_0805" V 9930 1550 50  0001 C CNN
 F 3 "" H 10000 1550 50  0000 C CNN
+F 4 "311-10KARCT-ND" V 10000 1550 60  0001 C CNN "MPN"
 	1    10000 1550
 	0    -1   -1   0
@@
 F 2 "Resistors_SMD:R_0805" V 9930 1700 50  0001 C CNN
 F 3 "" H 10000 1700 50  0000 C CNN
+F 4 "311-10KARCT-ND" V 10000 1700 60  0001 C CNN "MPN"
 	1    10000 1700
 	0    -1   -1   0
@@
 F 2 "Resistors_SMD:R_0805" V 9930 2000 50  0001 C CNN
 F 3 "" H 10000 2000 50  0000 C CNN
+F 4 "311-10KARCT-ND" V 10000 2000 60  0001 C CNN "MPN"
 	1    10000 2000
 	0    -1   -1   0
@@
 F 2 "Resistors_SMD:R_0805" V 9930 2150 50  0001 C CNN
 F 3 "" H 10000 2150 50  0000 C CNN
+F 4 "311-10KARCT-ND" V 10000 2150 60  0001 C CNN "MPN"
 	1    10000 2150
 	0    -1   -1   0
@@
 F 2 "Resistors_SMD:R_0805" V 9930 2350 50  0001 C CNN
 F 3 "" H 10000 2350 50  0000 C CNN
+F 4 "311-10KARCT-ND" V 10000 2350 60  0001 C CNN "MPN"
 	1    10000 2350
 	0    -1   -1   0
@@
 F 2 "Resistors_SMD:R_0805" V 9930 2500 50  0001 C CNN
 F 3 "" H 10000 2500 50  0000 C CNN
+F 4 "311-10KARCT-ND" V 10000 2500 60  0001 C CNN "MPN"
 	1    10000 2500
 	0    -1   -1   0
@@
 F 2 "Capacitors_SMD:C_0805" H 3200 1250 50  0001 C CNN
 F 3 "" H 3200 1250 50  0000 C CNN
+F 4 "CL21B103KBANNNC" H 3200 1250 60  0001 C CNN "MPN"
 	1    3200 1250
 	1    0    0    -1
@@
 F 2 "footprints:ARM_SWD_SMD" H 7400 4000 60  0001 C CNN
 F 3 "" H 7400 4000 60  0000 C CNN
+F 4 "20021121-00010C4LF" H 7700 4150 60  0001 C CNN "MPN"
 	1    7700 4150
 	1    0    0    -1
@@
 F 2 "Housings_SSOP:TSSOP-16_4.4x5mm_Pitch0.65mm" H 7100 2400 60  0001 C CNN
 F 3 "" H 7100 2400 60  0000 C CNN
+F 4 "TCA9546APWR" H 7100 2400 60  0001 C CNN "MPN"
 	1    7100 2400
 	1    0    0    -1
@@
 F 2 "Resistors_SMD:R_0805" V 3480 1850 50  0001 C CNN
 F 3 "" H 3550 1850 50  0000 C CNN
+F 4 "MCR10ERTJ000" V 3550 1850 60  0001 C CNN "MPN"
 	1    3550 1850
 	1    0    0    -1
