File: hw/relays/relays.kicad_pcb (KiCad board)
At the start: 2 copper layers, 38.1 x 16.5 mm, 8 parts, among them K1 EE2-3NU, P1 CONN_01X03, P2 CONN_01X02, P3 CONN_01X02, P4 CONN_01X02, Q1 MMBT3904

Commit message: Fix relay board after bad footprint fix
Parts:
- turned D1 to 270 degrees
Connections:
- P2 pad 1: /b_in -> /a_in
- P2 pad 2: /a_in -> /b_in
- P3 pad 1: /a_out_off -> /b_out_off
- P3 pad 2: /a_out_on -> /b_out_on
- P4 pad 1: /b_out_off -> /a_out_off
- P4 pad 2: /b_out_on -> /a_out_on
Routing:
- net VDD: track 17.6 -> 28.8 mm
- net /b_in: track 30.0 -> 35.4 mm
- net /a_in: track 35.4 -> 30.0 mm
- net Net-(D1-Pad2): track 10.3 -> 7.33 mm
