File: hw/relays/relays.sch (KiCad schematic (older format))
At the start: 8 parts, among them K1 EE2-3NU, P1 CONN_01X03, P2 CONN_01X02, P3 CONN_01X02, P4 CONN_01X02, Q1 MMBT3904

Commit message: Adding part numbers for relays board
Parts:
- D1: MPN (none) -> LL4148
- K1: MPN (none) -> EE2-3NU-L
- Q1: MPN (none) -> MMBT3904,215
- R1: MPN (none) -> RMCF0805JT1K00
Changed lines of the file:
@@
 F 2 "footprints:EE2-3NU" H 5550 1950 60  0001 C CNN
 F 3 "" H 5550 1950 60  0000 C CNN
+F 4 "EE2-3NU-L" H 5550 2400 60  0001 C CNN "MPN"
 	1    5550 2400
 	1    0    0    -1
@@
 F 2 "footprints:SOD-80" H 4200 2100 50  0001 C CNN
 F 3 "" H 4200 2100 50  0000 C CNN
+F 4 "LL4148" H 4200 2100 60  0001 C CNN "MPN"
 	1    4200 2100
 	0    1    1    0
@@
 F 2 "TO_SOT_Packages_SMD:SOT-23" H 4300 2725 50  0000 L CIN
 F 3 "" H 4100 2800 50  0000 L CNN
+F 4 "MMBT3904,215" H 4100 2800 60  0001 C CNN "MPN"
 	1    4100 2800
 	1    0    0    -1
@@
 F 2 "Resistors_SMD:R_0805" V 3530 2800 50  0001 C CNN
 F 3 "" H 3600 2800 50  0000 C CNN
+F 4 "RMCF0805JT1K00" V 3600 2800 60  0001 C CNN "MPN"
 	1    3600 2800
 	0    1    1    0

Commit message: Fix relay board after bad footprint fix
Connections:
- net a_in: now also P2.1 (P1); no longer P2.2 (P2)
- net a_out_off: now also P4.1 (P1); no longer P3.1 (P1)
- net a_out_on: now also P4.2 (P2); no longer P3.2 (P2)
- net b_in: now also P2.2 (P2); no longer P2.1 (P1)
- net b_out_off: now also P3.1 (P1); no longer P4.1 (P1)
- net b_out_on: now also P3.2 (P2); no longer P4.2 (P2)
Other:
- moved on the sheet: P3, P4
Changed lines of the file:
@@
 Text Label 4850 2600 0    60   ~ 0
 b_in
-Wire Wire Line
-	5950 2350 6750 2350
-Wire Wire Line
-	5950 2450 6750 2450
-Wire Wire Line
-	5950 2550 6750 2550
-Wire Wire Line
-	5950 2650 6750 2650
 Text Label 6300 2350 0    60   ~ 0
 a_out_off
@@
 L CONN_01X02 P3
 U 1 1 58744714
-P 6950 2400
-F 0 "P3" H 7100 2400 50  0000 C CNN
-F 1 "CONN_01X02" H 6950 2550 50  0000 C CNN
-F 2 "Pin_Headers:Pin_Header_Straight_1x02" H 6950 2400 50  0001 C CNN
-F 3 "" H 6950 2400 50  0000 C CNN
-	1    6950 2400
+P 6950 2600
+F 0 "P3" H 6950 2400 50  0000 C CNN
+F 1 "CONN_01X02" H 6950 3050 50  0000 C CNN
+F 2 "Pin_Headers:Pin_Header_Straight_1x02" H 6950 2600 50  0001 C CNN
+F 3 "" H 6950 2600 50  0000 C CNN
+	1    6950 2600
 	1    0    0    -1
 $EndComp
@@
 L CONN_01X02 P4
 U 1 1 58744775
-P 6950 2600
-F 0 "P4" H 7100 2600 50  0000 C CNN
-F 1 "CONN_01X02" H 6950 2400 50  0000 C CNN
-F 2 "Pin_Headers:Pin_Header_Straight_1x02" H 6950 2600 50  0001 C CNN
-F 3 "" H 6950 2600 50  0000 C CNN
-	1    6950 2600
+P 6950 2400
+F 0 "P4" H 6950 2550 50  0000 C CNN
+F 1 "CONN_01X02" H 6950 1950 50  0000 C CNN
+F 2 "Pin_Headers:Pin_Header_Straight_1x02" H 6950 2400 50  0001 C CNN
+F 3 "" H 6950 2400 50  0000 C CNN
+	1    6950 2400
 	1    0    0    -1
 $EndComp
@@
 $EndComp
 Text Label 3400 3400 0    60   ~ 0
+b_in
+Text Label 3400 3500 0    60   ~ 0
 a_in
-Text Label 3400 3500 0    60   ~ 0
-b_in
 $Comp
 L PWR_FLAG #FLG05
@@
 	0    1    1    0
 $EndComp
+Wire Wire Line
+	6750 2350 5950 2350
+Wire Wire Line
+	5950 2450 6750 2450
+Wire Wire Line
+	6750 2550 5950 2550
+Wire Wire Line
+	5950 2650 6750 2650
 $EndSCHEMATC
