File: hw/humidity/sht31_breakout.sch (KiCad schematic (older format))
At the start: 8 parts, among them P1 CONN_01X06, U1 SHT3x-DIS

Commit message: Made much smaller SHT31 breakout
We'll see if I can hand solder it...
Parts:
- removed P1: CONN_01X06, Pin_Headers:Pin_Header_Straight_1x06, symbol CONN_01X06
- removed R1, R4, R5: 10k, Capacitors_SMD:C_0603, symbol R
- added P1, P2: CONN_01X03, Pin_Headers:Pin_Header_Straight_1x03, symbol CONN_01X03
Connections:
- net ALERT: now also P1.3 (P3)
- net GND: now also P1.1 (P1)
- net SCL: now also P2.2 (P2)
- net SDA: now also P1.2 (P2)
- net VDD: now also P2.1 (P1)
- net nRESET: now also P2.3 (P3)
Changed lines of the file:
@@
-$EndComp
-$Comp
-L R R4
-U 1 1 582131B6
-P 1500 3100
-F 0 "R4" V 1580 3100 50  0000 C CNN
-F 1 "10k" V 1500 3100 50  0000 C CNN
-F 2 "Capacitors_SMD:C_0603" V 1430 3100 50  0001 C CNN
-F 3 "" H 1500 3100 50  0000 C CNN
-	1    1500 3100
-	1    0    0    -1
-$EndComp
-$Comp
-L R R1
-U 1 1 582131D5
-P 1250 3100
-F 0 "R1" V 1330 3100 50  0000 C CNN
-F 1 "10k" V 1250 3100 50  0000 C CNN
-F 2 "Capacitors_SMD:C_0603" V 1180 3100 50  0001 C CNN
-F 3 "" H 1250 3100 50  0000 C CNN
-	1    1250 3100
-	1    0    0    -1
-$EndComp
-$Comp
-L R R5
-U 1 1 582131FC
-P 1800 3100
-F 0 "R5" V 1880 3100 50  0000 C CNN
-F 1 "10k" V 1800 3100 50  0000 C CNN
-F 2 "Capacitors_SMD:C_0603" V 1730 3100 50  0001 C CNN
-F 3 "" H 1800 3100 50  0000 C CNN
-	1    1800 3100
-	1    0    0    -1
 $EndComp
 $Comp
@@
 	3350 2100 2950 2100
 Wire Wire Line
-	3350 2400 2950 2400
+	2950 2400 3350 2400
 Wire Wire Line
 	3350 2300 3250 2300
@@
 $EndComp
 Wire Wire Line
-	1500 2100 1500 1900
+	1500 1900 1500 2100
 Wire Wire Line
-	1500 2500 1500 2400
+	1500 2400 1500 2500
 Wire Wire Line
-	1500 1600 1500 1500
+	1500 1500 1500 1600
 $Comp
 L VDD #PWR02
@@
 ADDR
 Wire Wire Line
-	1250 2950 1800 2950
-Connection ~ 1500 2950
+	3700 3350 3300 3350
 Wire Wire Line
-	1800 3250 1800 3350
+	3700 3450 3300 3450
 Wire Wire Line
-	1800 3350 2100 3350
+	3700 2950 3300 2950
 Wire Wire Line
-	1500 3250 1500 3500
+	3700 2850 3300 2850
 Wire Wire Line
-	1500 3500 2100 3500
-Text Label 1350 2950 0    60   ~ 0
+	3700 3550 3300 3550
+Wire Wire Line
+	3700 3050 3300 3050
+Text Label 3300 3350 0    60   ~ 0
 VDD
-Text Label 2100 3350 0    60   ~ 0
+Text Label 3300 3450 0    60   ~ 0
+SCL
+Text Label 3300 2950 0    60   ~ 0
 SDA
-Text Label 2100 3500 0    60   ~ 0
-SCL
-Wire Wire Line
-	1250 3250 1250 3650
-Wire Wire Line
-	1250 3650 2100 3650
-Text Label 2100 3650 0    60   ~ 0
+Text Label 3300 2850 0    60   ~ 0
+VSS
+Text Label 3300 3550 0    60   ~ 0
 nRESET
-$Comp
-L CONN_01X06 P1
-U 1 1 582140C4
-P 3800 3100
-F 0 "P1" H 3800 3450 50  0000 C CNN
-F 1 "CONN_01X06" V 3900 3100 50  0000 C CNN
-F 2 "Pin_Headers:Pin_Header_Straight_1x06" H 3800 3100 50  0001 C CNN
-F 3 "" H 3800 3100 50  0000 C CNN
-	1    3800 3100
-	1    0    0    -1
-$EndComp
-Wire Wire Line
-	3600 2850 3200 2850
-Wire Wire Line
-	3600 2950 3200 2950
-Wire Wire Line
-	3600 3050 3200 3050
-Wire Wire Line
-	3600 3150 3200 3150
-Wire Wire Line
-	3600 3250 3200 3250
-Wire Wire Line
-	3600 3350 3200 3350
-Text Label 3200 2850 0    60   ~ 0
-VDD
-Text Label 3200 2950 0    60   ~ 0
-SCL
-Text Label 3200 3050 0    60   ~ 0
-SDA
-Text Label 3200 3150 0    60   ~ 0
-VSS
-Text Label 3200 3250 0    60   ~ 0
-nRESET
-Text Label 3200 3350 0    60   ~ 0
+Text Label 3300 3050 0    60   ~ 0
 ALERT
 $Comp
@@
 Wire Wire Line
 	1100 2150 1100 2450
+$Comp
+L CONN_01X03 P1
+U 1 1 5892AA7E
+P 3900 2950
+F 0 "P1" H 3900 3150 50  0000 C CNN
+F 1 "CONN_01X03" V 4000 2950 50  0000 C CNN
+F 2 "Pin_Headers:Pin_Header_Straight_1x03" H 3900 2950 50  0001 C CNN
+F 3 "" H 3900 2950 50  0000 C CNN
+	1    3900 2950
+	1    0    0    -1
+$EndComp
+$Comp
+L CONN_01X03 P2
+U 1 1 5892AB09
+P 3900 3450
+F 0 "P2" H 3900 3650 50  0000 C CNN
+F 1 "CONN_01X03" V 4000 3450 50  0000 C CNN
+F 2 "Pin_Headers:Pin_Header_Straight_1x03" H 3900 3450 50  0001 C CNN
+F 3 "" H 3900 3450 50  0000 C CNN
+	1    3900 3450
+	1    0    0    -1
+$EndComp
 $EndSCHEMATC

Commit message: Start designing flex pcb :D
Parts:
- removed P1, P2: CONN_01X03, Pin_Headers:Pin_Header_Straight_1x03, symbol CONN_01X03
- added J1: CONN_01X04, footprints:smd_flex_4, symbol CONN_01X04
Connections:
- net nRESET is gone; now on net VDD: U1.6 (nRESET)
- net GND: now also J1.1 (P1)
- net SCL: now also J1.4 (P4)
- net SDA: now also J1.3 (P3)
- net VDD: now also J1.2 (P2)
- net ALERT: no longer names the net of U1.3 (ALERT)
- no-connect marks 0 -> 1
Changed lines of the file:
@@
 Wire Wire Line
 	3350 1800 2950 1800
-Wire Wire Line
-	3350 1900 2950 1900
-Wire Wire Line
-	3350 2200 2950 2200
 Text Label 2950 1800 0    60   ~ 0
 ADDR
-Text Label 2950 1900 0    60   ~ 0
-ALERT
-Text Label 2950 2200 0    60   ~ 0
-nRESET
 $Comp
 L GND #PWR01
@@
 ADDR
 Wire Wire Line
-	3700 3350 3300 3350
+	4200 2950 3800 2950
 Wire Wire Line
-	3700 3450 3300 3450
+	4200 3150 3800 3150
 Wire Wire Line
-	3700 2950 3300 2950
+	4200 3050 3800 3050
 Wire Wire Line
-	3700 2850 3300 2850
-Wire Wire Line
-	3700 3550 3300 3550
-Wire Wire Line
-	3700 3050 3300 3050
-Text Label 3300 3350 0    60   ~ 0
+	4200 2850 3800 2850
+Text Label 3800 2950 0    60   ~ 0
 VDD
-Text Label 3300 3450 0    60   ~ 0
+Text Label 3800 3150 0    60   ~ 0
 SCL
-Text Label 3300 2950 0    60   ~ 0
+Text Label 3800 3050 0    60   ~ 0
 SDA
-Text Label 3300 2850 0    60   ~ 0
+Text Label 3800 2850 0    60   ~ 0
 VSS
-Text Label 3300 3550 0    60   ~ 0
-nRESET
-Text Label 3300 3050 0    60   ~ 0
-ALERT
 $Comp
 L C C1
@@
 	1100 2150 1100 2450
 $Comp
-L CONN_01X03 P1
-U 1 1 5892AA7E
-P 3900 2950
-F 0 "P1" H 3900 3150 50  0000 C CNN
-F 1 "CONN_01X03" V 4000 2950 50  0000 C CNN
-F 2 "Pin_Headers:Pin_Header_Straight_1x03" H 3900 2950 50  0001 C CNN
-F 3 "" H 3900 2950 50  0000 C CNN
-	1    3900 2950
+L CONN_01X04 J1
+U 1 1 596A2ADA
+P 4400 3000
+F 0 "J1" H 4400 3250 50  0000 C CNN
+F 1 "CONN_01X04" V 4500 3000 50  0000 C CNN
+F 2 "footprints:smd_flex_4" H 4400 3000 50  0001 C CNN
+F 3 "" H 4400 3000 50  0001 C CNN
+	1    4400 3000
 	1    0    0    -1
 $EndComp
-$Comp
-L CONN_01X03 P2
-U 1 1 5892AB09
-P 3900 3450
-F 0 "P2" H 3900 3650 50  0000 C CNN
-F 1 "CONN_01X03" V 4000 3450 50  0000 C CNN
-F 2 "Pin_Headers:Pin_Header_Straight_1x03" H 3900 3450 50  0001 C CNN
-F 3 "" H 3900 3450 50  0000 C CNN
-	1    3900 3450
-	1    0    0    -1
-$EndComp
+NoConn ~ 3350 1900
+Wire Wire Line
+	3350 2200 3250 2200
+Wire Wire Line
+	3250 2200 3250 2100
+Connection ~ 3250 2100
 $EndSCHEMATC

Commit message: Updated sht31 breakout to be wedge shaped!
Parts:
- J1: footprint footprints:smd_flex_4 -> Pin_Headers:Pin_Header_Straight_1x04_Pitch2.54mm
Changed lines of the file:
@@
 F 0 "J1" H 4400 3250 50  0000 C CNN
 F 1 "CONN_01X04" V 4500 3000 50  0000 C CNN
-F 2 "footprints:smd_flex_4" H 4400 3000 50  0001 C CNN
+F 2 "Pin_Headers:Pin_Header_Straight_1x04_Pitch2.54mm" H 4400 3000 50  0001 C CNN
 F 3 "" H 4400 3000 50  0001 C CNN
 	1    4400 3000
